Commit message: OWRS-130 #time 45m Getting closer. All the parts are there now, just need to line them up properly

File: rover/src/owr_bluetounge_tf/robots/ForHarryForROSVersB.URDF (robot description, URDF)
Before this commit: robot owr_bluetounge_tf, 5 links, 4 joints
Links:
- added link Bogey, mass 2.3410771686329; collision mesh filename=package://owr_bluetounge_tf/meshes/Bogey.STL; visual mesh filename=package://owr_bluetounge_tf/meshes/Bogey.STL
Joints:
- removed joint base_to_right_leg
- added joint base_to_bogey: type fixed, parent base_link, child Bogey, origin xyz=.2 0 0 rpy=0 0 1.5, axis 0 0 1
- added joint base_to_notwheels: type fixed, parent Bogey, child NotWheels

Commit message: OWRS-130 #time 30m moving joints

File: rover/src/owr_bluetounge_tf/robots/ForHarryForROSVersB.URDF (robot description, URDF)
Before this commit: robot owr_bluetounge_tf, 5 links, 4 joints
Joints:
- joint AAxle: axis 0 0 0 -> 0 0 1; type fixed -> continuous
- joint BAxle: axis 0 0 0 -> 0 0 1; type fixed -> continuous
- joint CAxle: axis 0 0 0 -> 0 0 1; type fixed -> continuous

Commit message: OWRS-130 #time 30m Bogey lined up, but wheel modules won't align :(

File: rover/src/owr_bluetounge_tf/robots/ForHarryForROSVersB.URDF (robot description, URDF)
Before this commit: robot owr_bluetounge_tf, 6 links, 5 joints
Joints:
- joint base_to_notwheels: origin (none) -> xyz=0 -0.05 -0.17

Commit message: OWRS-130 #time 5m

File: rover/src/owr_bluetounge_tf/robots/ForHarryForROSVersB.URDF (robot description, URDF)
Before this commit: robot owr_bluetounge_tf, 6 links, 5 joints
Links:
- removed link AWheel
- removed link BWheel
- removed link Bogey
- removed link CWheel
- removed link NotWheels
- added link BogeyL, mass 2.3410771686329; collision mesh filename=package://owr_bluetounge_tf/meshes/Bogey.STL; visual mesh filename=package://owr_bluetounge_tf/meshes/Bogey.STL
- added link WheelLF, mass 1.86318344508723; collision mesh filename=package://owr_bluetounge_tf/meshes/Wheel.STL; visual mesh filename=package://owr_bluetounge_tf/meshes/Wheel.STL
- added link WideWheelBaseLF, mass 2.724043620833; collision mesh filename=package://owr_bluetounge_tf/meshes/WideWheelBase.STL; visual mesh filename=package://owr_bluetounge_tf/meshes/WideWheelBase.STL
Joints:
- removed joint AAxle
- removed joint BAxle
- removed joint CAxle
- removed joint base_to_notwheels
- added joint Axle: type fixed, parent WideWheelBaseLF, child WheelLF, origin xyz=0.0254710786476053 -0.0201166854458847 0.000315728425903225 rpy=1.5707963267949 0 0, axis 0 0 0
- added joint lf_to_bogey: type fixed, parent BogeyL, child WideWheelBaseLF, origin xyz=0 0 -.33 rpy=0 0 0, axis 0 0 0
- joint base_to_bogey: child Bogey -> BogeyL
