Commit message: OWRS-139 #time 30m urdf good, localization probably shouldn't use though

File: rover/src/owr_bluetounge_tf/robots/bluetounge.URDF (robot description, URDF)
Before this commit: robot bluetounge, 13 links, 12 joints
Joints:
- joint base_to_right_bogey: origin xyz=-.3 0 0.027 rpy=0 3.14159265 4.71238898 -> xyz=-.4 0 0.027 rpy=0 3.14159265 4.71238898

Commit message: OWRS-130 #time 30m Hokuyo tfs and a few other things

File: rover/src/owr_bluetounge_tf/robots/bluetounge.URDF (robot description, URDF)
Before this commit: robot bluetounge, 13 links, 12 joints
Links:
- added link laser, mass 1e-5; collision box size=0.1 0.1 0.1; visual mesh filename=package://owr_bluetounge_tf/meshes/hokuyo.dae
Joints:
- added joint hokuyo_joint: type fixed, parent base_link, child laser, origin xyz=0 .3 0 rpy=0 0 0, axis 0 0 0

Commit message: OWRS-71 #In Progress #time 1h 30m  should working

File: rover/src/owr_bluetounge_tf/robots/bluetounge.URDF (robot description, URDF)
Before this commit: robot bluetounge, 14 links, 13 joints
Joints:
- joint hokuyo_joint: origin xyz=0 .3 0 rpy=0 0 0 -> xyz=0 .3 0.1 rpy=0 0 0

Commit message: URDF

File: rover/src/owr_bluetounge_tf/robots/bluetounge.URDF (robot description, URDF)
Before this commit: robot bluetounge, 14 links, 13 joints
Joints:
- joint hokuyo_joint: origin xyz=0 .3 0.1 rpy=0 0 0 -> xyz=0 .3 -0.1 rpy=0 3.14159 0

Commit message: OWRS-73 #time 2h

File: rover/src/owr_bluetounge_tf/robots/bluetounge.URDF (robot description, URDF)
Before this commit: robot bluetounge, 14 links, 13 joints
Joints:
- joint hokuyo_joint: origin xyz=0 .3 -0.1 rpy=0 3.14159 0 -> xyz=-0.075 .3 -0.1 rpy=0 3.14159 0

Commit message: OWRS-73 #time 1h urdf has lidar in correct position

File: rover/src/owr_bluetounge_tf/robots/bluetounge.URDF (robot description, URDF)
Before this commit: robot bluetounge, 14 links, 13 joints
Joints:
- joint hokuyo_joint: origin xyz=-0.075 .3 -0.1 rpy=0 3.14159 0 -> xyz=-0.075 -.245 -0.1 rpy=0 3.14159 3.14159

Commit message: Tf and other fixes

File: rover/src/owr_bluetounge_tf/robots/bluetounge.URDF (robot description, URDF)
Before this commit: robot bluetounge, 14 links, 13 joints
Joints:
- joint hokuyo_joint: origin xyz=-0.075 -.245 -0.1 rpy=0 3.14159 3.14159 -> xyz=-0.075 -.245 0.1 rpy=0 3.14159 1.57079633

Commit message: tf

File: rover/src/owr_bluetounge_tf/robots/bluetounge.URDF (robot description, URDF)
Before this commit: robot bluetounge, 14 links, 13 joints
Joints:
- joint hokuyo_joint: origin xyz=-0.075 -.245 0.1 rpy=0 3.14159 1.57079633 -> xyz=0.075 -.245 -0.1 rpy=0 3.14159 1.57079633
