Commit message: OWRS-179 3d-model OWRS-97 #time 1h appears to be working urdf model for the simulator

File: rover/src/owr_bluetounge_tf/robots/owr_bluetounge_tf.URDF (robot description, URDF)
Before this commit: robot owr_bluetounge_tf, 28 links, 27 joints
Links:
- link middle_left_wheel: geometry collision mesh filename=package://owr_bluetounge_tf/meshes/back_left_wheel.STL; visual mesh filename=package://owr_bluetounge_tf/meshes/back_left_wheel.STL
Joints:
- joint back_left_wheel_axel: axis 0 0 0 -> 0 0 1; origin xyz=-0.0254000000000002 -0.0235 0.01363 rpy=3.14159265358979 0 0 -> xyz=-0.0254000000000002 0.0235 0.26363 rpy=3.14159265358979 0 0; type fixed -> continuous
- joint back_right_bogey_axel: origin xyz=0.714828885819377 -0.161773416923871 0.373659999999994 rpy=2.14755054093466 -1.5707963267949 0 -> xyz=0.714828885819377 -0.161773416923871 0.373659999999994 rpy=2.14755054093466 -1.5707963267949 3.14159265359
- joint back_right_wheel_axel: axis 0 0 0 -> 1 0 0; type fixed -> continuous
- joint front_left_wheel_axel: axis 0 0 0 -> 0 0 1; origin xyz=0.00399999999999995 0.0290000000000001 -0.0253999999999999 rpy=3.14159265358979 -1.5707963267949 0 -> xyz=-0.25399999999999995 0.0290000000000001 -0.0253999999999999 rpy=0 1.57079632679 0 ; type fixed -> continuous
- joint front_right_wheel_axel: axis 0 0 0 -> 1 0 0; type fixed -> continuous
- joint middle_left_wheel_axel: axis 0 0 0 -> 0 0 1; origin xyz=-0.0254000000000002 -0.0235 0.01363 rpy=3.14159265358979 0 0 -> xyz=0.4754000000000002 0.0235 0.26363 rpy=3.14159265358979 0 0; type fixed -> continuous
- joint middle_right_wheel_axel: axis 0 0 0 -> 1 0 0; type fixed -> continuous

Commit message: OWRS-79 #time 3h added lidar tilt and a proper lidar urdf. When we do this on the new bluetounge should make sure that the CAD for the tilt is in a horizontal position so it is easier to align the lidar

File: rover/src/owr_bluetounge_tf/robots/owr_bluetounge_tf.URDF (robot description, URDF)
Before this commit: robot owr_bluetounge_tf, 30 links, 29 joints
Links:
- removed link laser
- added link laser_tilt_base, mass 0.060913; collision mesh filename=package://owr_bluetounge_tf/meshes/laser_tilt_base.STL; visual mesh filename=package://owr_bluetounge_tf/meshes/laser_tilt_base.STL
- added link laser_tilt_tilt, mass 0.060855; collision mesh filename=package://owr_bluetounge_tf/meshes/laser_tilt_tilt.STL; visual mesh filename=package://owr_bluetounge_tf/meshes/laser_tilt_tilt.STL
Joints:
- removed joint hokuyo_joint
- added joint laser_tilt_base_link: type fixed, parent base_link, child laser_tilt_base, origin xyz=.245 0.28 0.145  rpy=0.785398 0 -1.5708, axis 0 0 0
- added joint laser_tilt_joint: type continuous, parent laser_tilt_base, child laser_tilt_tilt, origin xyz=0.3929 -0.01446 -0.014263 rpy=0.82137 0 0, axis -1 0 0

Commit message: OWRS-79 #time 1h 30m got gazebo working properly. Managed to drive rover in a straight line, but it does backflips if you try to turn. (This may be due to: incorrect inertia data from solidworks, not having the bogey fixed with the metal rods, and/or not allowing the bogey axels to rotate)

File: rover/src/owr_bluetounge_tf/robots/owr_bluetounge_tf.URDF (robot description, URDF)
Before this commit: robot owr_bluetounge_tf, 31 links, 30 joints
Links:
- added link robot_base, mass 8.39051518849641; collision mesh filename=package://owr_bluetounge_tf/meshes/base_link.STL; visual mesh filename=package://owr_bluetounge_tf/meshes/base_link.STL
- link base_link: mass 8.39051518849641 -> None; geometry 
- link camera0: mass 1e-5 -> 0.10277; geometry collision mesh filename=package://owr_bluetounge_tf/meshes/camera.STL; visual mesh filename=package://owr_bluetounge_tf/meshes/camera.STL
Joints:
- removed joint laser_tilt_base_link
- added joint base_link_joint: type fixed, parent base_link, child robot_base, origin xyz=0 0 0  rpy=0 0 0, axis 0 0 0
- added joint laser_tilt_robot_base: type fixed, parent robot_base, child laser_tilt_base, origin xyz=.245 0.28 0.145  rpy=0.785398 0 -1.5708, axis 0 0 0
- joint camera0_joint: axis 0 1 0 -> 0 0 0; origin xyz=0 1 0 rpy=0 0 0 -> xyz=1.9 0.1 0.12 rpy=${90 * (PI/180)} ${180 * (PI/180)} 0; parent base_link -> robot_base
- joint lazy_susan: parent base_link -> robot_base
- joint left_axel: parent base_link -> robot_base
- joint right_axel: parent base_link -> robot_base

Commit message: OWRS-97 #time 2h got camera model with correct origin and other fixes

File: rover/src/owr_bluetounge_tf/robots/owr_bluetounge_tf.URDF (robot description, URDF)
Before this commit: robot owr_bluetounge_tf, 32 links, 31 joints
Joints:
- joint camera0_joint: origin xyz=1.9 0.1 0.12 rpy=${90 * (PI/180)} ${180 * (PI/180)} 0 -> xyz=0.2 0.2 0.12 rpy=0 0 0

Commit message: branch cleanup

File: rover/src/owr_bluetounge_tf/robots/owr_bluetounge_tf.URDF (robot description, URDF)
Before this commit: robot owr_bluetounge_tf, 28 links, 27 joints
Links:
- removed link arm_fibbia
- removed link arm_lazy_susan
- removed link arm_lower
- removed link arm_tibbia
- removed link arm_triangle
- removed link arm_upper_plate
- removed link back_left_bogey
- removed link back_left_wheel
- removed link back_right_bogey
- removed link back_right_wheel
- removed link claw_base
- removed link claw_clamp_right
- removed link claw_gear_right
- removed link claw_left_gear
- removed link claw_left_grip
- removed link claw_r_clip
- removed link claw_wrist
- removed link front_left_wheel
- removed link front_right_wheel
- removed link left_bogey
- removed link linear_base_top
- removed link linear_bottom
- removed link linear_bottom_top
- removed link linear_top_top
- removed link middle_left_wheel
- removed link middle_right_wheel
- removed link right_bogey
- added link left_linear_base, mass 22.0243812744452; collision mesh filename=package://owr_bluetounge_tf/meshes/left_linear_base.STL; visual mesh filename=package://owr_bluetounge_tf/meshes/left_linear_base.STL
- added link left_linear_shaft, mass 23.1723954465805; collision mesh filename=package://owr_bluetounge_tf/meshes/left_linear_shaft.STL; visual mesh filename=package://owr_bluetounge_tf/meshes/left_linear_shaft.STL
- added link long_link, mass 18.642477796077; collision mesh filename=package://owr_bluetounge_tf/meshes/long_link.STL; visual mesh filename=package://owr_bluetounge_tf/meshes/long_link.STL
- added link long_link2, mass 18.642477796077; collision mesh filename=package://owr_bluetounge_tf/meshes/long_link2.STL; visual mesh filename=package://owr_bluetounge_tf/meshes/long_link2.STL
- added link right_linear_base, mass 22.0243812744452; collision mesh filename=package://owr_bluetounge_tf/meshes/right_linear_base.STL; visual mesh filename=package://owr_bluetounge_tf/meshes/right_linear_base.STL
- added link right_linear_shaft, mass 23.1723954465805; collision mesh filename=package://owr_bluetounge_tf/meshes/right_linear_shaft.STL; visual mesh filename=package://owr_bluetounge_tf/meshes/right_linear_shaft.STL
- link base_link: mass 8.39051518849641 -> 11.142477796077
Joints:
- removed joint arm_fibbia_actuator_joint
- removed joint arm_lower_joint
- removed joint arm_tibbia_joint
- removed joint arm_triangle
- removed joint arm_upper_plate_joint
- removed joint back_left_bogey_axel
- removed joint back_left_wheel_axel
- removed joint back_right_bogey_axel
- removed joint back_right_wheel_axel
- removed joint claw_base_joint
- removed joint claw_clamp_right
- removed joint claw_gear_right
- removed joint claw_left_gear
- removed joint claw_left_grip
- removed joint claw_r_clip
- removed joint claw_wrist_rotate
- removed joint front_left_wheel_axel
- removed joint front_right_wheel_axel
- removed joint lazy_susan
- removed joint left_axel
- removed joint linear_actuator_top
- removed joint linear_bottom_joint
- removed joint linear_bottom_rotate
- removed joint middle_left_wheel_axel
- removed joint middle_right_wheel_axel
- removed joint right_axel
- removed joint top_linear_rotate
- added joint left_linear_base_rotate: type continuous, parent base_link, child left_linear_base, origin xyz=-0.400000000000018 0 -0.0249999999999806 rpy=-1.5707963267949 0.0556932148995094 -1.49498600701826E-14, axis 0 0 -1
- added joint left_linear_extension: type prismatic, parent left_linear_base, child left_linear_shaft, origin xyz=0 0.20488 0 rpy=-3.9443E-31 0 1.3184E-16, axis 0 1 0, limit lower=0 upper=1 effort=1000 velocity=1000
- added joint left_linear_shaft_rotate: type continuous, parent left_linear_shaft, child long_link, origin xyz=0 0.7 0 rpy=-1.1427E-16 -1.3215E-16 -0.13669, axis 0 0 -1
- added joint right_linear_base_rotate: type continuous, parent base_link, child right_linear_base, origin xyz=0.40000000000003 0 -0.0249999999992338 rpy=-1.5707963267949 -0.5088897326569 -5.55111512448809E-17, axis 0 0 -1
- added joint right_linear_extension: type prismatic, parent right_linear_base, child right_linear_shaft, origin xyz=0 0.21412 0 rpy=6.6296E-27 -2.8208E-30 1.6653E-16, axis 0 1 0, limit lower=0 upper=1 effort=1000 velocity=1000
- added joint right_linear_shaft_rotate: type continuous, parent right_linear_shaft, child long_link2, origin xyz=0 0.699999999996918 0 rpy=-1.19874294786595E-15 1.47299632878217E-14 0.427890034635904, axis 0 0 -1

Commit message: OWRS-156 #time 2h transforms proof of concept working, main code in ArmWidgetGUI.cpp

File: rover/src/owr_bluetounge_tf/robots/owr_bluetounge_tf.URDF (robot description, URDF)
Before this commit: robot owr_bluetounge_tf, 7 links, 6 joints
Links:
- removed link left_linear_base
- removed link left_linear_shaft
- removed link long_link
- removed link long_link2
- removed link right_linear_base
- removed link right_linear_shaft
- added link bottom_actuator_base, mass 0.529218600966516; collision mesh filename=package://owr_bluetounge_tf/meshes/bottom_actuator_base.STL; visual mesh filename=package://owr_bluetounge_tf/meshes/bottom_actuator_base.STL
- added link bottom_actuator_shaft, mass 0.834414950203527; collision mesh filename=package://owr_bluetounge_tf/meshes/bottom_actuator_shaft.STL; visual mesh filename=package://owr_bluetounge_tf/meshes/bottom_actuator_shaft.STL
- added link end_plate, mass 0.0752794153885444; collision mesh filename=package://owr_bluetounge_tf/meshes/end_plate.STL; visual mesh filename=package://owr_bluetounge_tf/meshes/end_plate.STL
- added link rocker, mass 0.441329423356222; collision mesh filename=package://owr_bluetounge_tf/meshes/rocker.STL; visual mesh filename=package://owr_bluetounge_tf/meshes/rocker.STL
- added link structural_main, mass 0.54398717386464; collision mesh filename=package://owr_bluetounge_tf/meshes/structural_main.STL; visual mesh filename=package://owr_bluetounge_tf/meshes/structural_main.STL
- added link sync_main, mass 0.648821763310334; collision mesh filename=package://owr_bluetounge_tf/meshes/sync_main.STL; visual mesh filename=package://owr_bluetounge_tf/meshes/sync_main.STL
- added link sync_minor, mass 0.246647562813028; collision mesh filename=package://owr_bluetounge_tf/meshes/sync_minor.STL; visual mesh filename=package://owr_bluetounge_tf/meshes/sync_minor.STL
- added link sync_plate, mass 0.109130569272771; collision mesh filename=package://owr_bluetounge_tf/meshes/sync_plate.STL; visual mesh filename=package://owr_bluetounge_tf/meshes/sync_plate.STL
- added link top_actuator_base, mass 0.500146440873381; collision mesh filename=package://owr_bluetounge_tf/meshes/top_actuator_base.STL; visual mesh filename=package://owr_bluetounge_tf/meshes/top_actuator_base.STL
- added link top_actuator_shaft, mass 0.707194764725093; collision mesh filename=package://owr_bluetounge_tf/meshes/top_actuator_shaft.STL; visual mesh filename=package://owr_bluetounge_tf/meshes/top_actuator_shaft.STL
- link base_link: mass 11.142477796077 -> 0.684098692441384
Joints:
- removed joint left_linear_base_rotate
- removed joint left_linear_extension
- removed joint left_linear_shaft_rotate
- removed joint right_linear_base_rotate
- removed joint right_linear_extension
- removed joint right_linear_shaft_rotate
- added joint base_to_structural_main: type continuous, parent base_link, child structural_main, origin xyz=-0.0275200000000058 0 0.0289999999999882 rpy=1.5707963267949 -1.04097774036042 3.14159265358979, axis 0 0 1
- added joint bottom_actuator_base_rotate: type continuous, parent structural_main, child bottom_actuator_base, origin xyz=0 0.0880000000000138 -0.0320000000000025 rpy=2.10061491322937 -1.5707963267949 0, axis -1 0 0
- added joint bottom_actuator_extension: type prismatic, parent bottom_actuator_base, child bottom_actuator_shaft, origin xyz=0.032 0.21857 -0.11088 rpy=-1.5708 -1.1013 1.5708, axis 0 1 0, limit lower=-10 upper=10 effort=1000 velocity=1000
- added joint structural_main_to_sync_plate: type continuous, parent structural_main, child sync_plate, origin xyz=0.600097477062092 -0.0215765064114193 -0.0380000000000022 rpy=6.88704600198579E-17 1.01259404278687E-16 2.16806796081584, axis 0 0 -1
- added joint sync_minor_to_end_plate: type continuous, parent sync_minor, child end_plate, origin xyz=0.439282685338784 -0.017880203257983 -0.00399999999999935 rpy=0 0 1.8863672273632, axis 0 0 -1
- added joint sync_plate_to_rocker: type continuous, parent structural_main, child rocker, origin xyz=0.534024000000006 0 -0.0179999999999996 rpy=3.14159265358979 9.70332217454327E-17 0.914672033584322, axis 0 0 1
- added joint sync_plate_to_sync_minor: type continuous, parent sync_plate, child sync_minor, origin xyz=0 0 0 rpy=3.14159265358979 0 1.88517119022756, axis 0 0 -1
- added joint top_actuator_base_rotate: type continuous, parent base_link, child top_actuator_base, origin xyz=0.0898381894927384 0 0.209155716713238 rpy=1.14619501972752 5.59161451734894E-09 1.57079633916291, axis 1 0 0
- added joint top_actuator_extension: type prismatic, parent top_actuator_base, child top_actuator_shaft, origin xyz=0 0.072106 0 rpy=3.1415 -1.5708 -3.1415, axis 0 1 0, limit lower=-10 upper=10 effort=1000 velocity=1000
- added joint top_actuator_to_sync_main: type continuous, parent top_actuator_shaft, child sync_main, origin xyz=-0.115124184387589 -0.175473958284494 -0.0419999999999976 rpy=3.14159265358979 0 1.67149338911103, axis 0 0 -1
