Commit message: OWRS-130 #time 30m all the wheels on one side of the bogey

File: rover/src/RightBogey/robots/Version A (With Wheels).SLDASM.URDF (robot description, URDF)
Before this commit: robot RightBogey, 7 links, 6 joints
Joints:
- joint AxleRB: axis 0 0 0 -> 1 0 0; origin xyz=-0.02 .16 0.000315728425903225 rpy=1.5707963267949 0 0 -> xyz=0 0.5 0.02 rpy=1.5707963267949 0 0
- joint AxleRM: axis 0 0 0 -> 1 0 0; origin xyz=-0.02 .16 0.000315728425903225 rpy=1.5707963267949 0 0 -> xyz=0 0.02 0.02 rpy=1.5707963267949 0 0
