Commit message: OWRS-204 #time 2h finally got a working, valid simulation model that can be used to test steering. Need to confirm gazebo setup, but should be #done

File: rover/src/owr_bluetounge2_tf/robots/owr_bluetounge2_tf-old.URDF (robot description, URDF)
Before this commit: robot owr_bluetounge2_tf, 53 links, 52 joints
Links:
- removed link back_right_swerve_top
- removed link front_right_swerve_top
- link arm_bottom_actuator_base: mass 0.5292185810438 -> 0.529218581187352
- link arm_bottom_actuator_shaft: mass 0.834414953724231 -> 0.834414953724234
- link arm_bottom_plates: mass 0.523833534252721 -> 0.523833534252722
- link arm_lower_bottom_plates: mass 0.421175783744303 -> 0.421175783744302
- link arm_lower_top_plates: mass 0.222440263368329 -> 0.222440263368328
- link arm_top_actuator_base: mass 0.505108099872299 -> 0.50510809979627
- link arm_top_actuator_shaft: mass 0.707194769757707 -> 0.707194769757711
- link back_right_springs: mass 0.0728462856892432 -> 0.0728462856892431
- link back_right_swerve_axel: mass 2.34386977405423 -> 2.39145632608747; geometry collision mesh filename=package://owr_bluetounge2_tf/meshes/back_right_swerve_axel.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; visual mesh filename=package://owr_bluetounge2_tf/meshes/back_right_swerve_axel.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
- link back_right_wheel: geometry collision mesh filename=package://owr_bluetounge2_tf/meshes/back_right_wheel.STL; visual mesh filename=package://owr_bluetounge2_tf/meshes/back_right_wheel.STL
- link claw_base: mass 0.0771754639307836 -> 0.0771754639307835
- link claw_left: mass 0.0196972369456186 -> 0.0196972369456185
- link claw_wrist: mass 0.0918795943669829 -> 0.0918795943669828
- link front_left_swerve_axel: mass 2.36761790939096 -> 2.3676
- link front_right_leg_base: mass 0.0851788397766331 -> 0.0851788397766332
Joints:
- removed joint back_right_swerve_to_suspension
- removed joint front_right_swerve_to_suspension
- joint arm_bottom_actuator: axis -0.0880363362662565 0.996117263928708 0 -> -0.088036 0.99612 0; origin xyz=0.0320003944226702 0.0808917432002021 -0.0448335334962513 rpy=-1.57079632679491 -1.06470265084296 1.57079632679491 -> xyz=0.032 0.080892 -0.044834 rpy=-1.5708 -1.0647 1.5708
- joint arm_bottom_actuator_base_rotate: origin xyz=0 0.0879999874476814 -0.0579999944206897 rpy=0.00603226555870947 -1.57079631189374 -1.14785595903188 -> xyz=0 0.0880000012352829 -0.0580000000598536 rpy=2.00092816923768 -1.5707963267949 0
- joint arm_bottom_plates_rotate: origin xyz=0.0275184794744797 -0.0259999999999933 0.153127996289484 rpy=1.57079632679489 -1.14066443094574 1.37649429779348E-13 -> xyz=0.0275184819386707 -0.0259999999999941 0.153128001655061 rpy=1.57079632679489 -1.14066448437714 1.40494955389075E-13
- joint arm_lower_bottom_plates_rotate: origin xyz=-0.0472198179654527 0.446676991521919 -0.0219995999980216 rpy=1.2490009027033E-16 -8.32667268468867E-17 -0.834690804163616 -> xyz=-0.0472197994353847 0.446676986623695 -0.0219995999980227 rpy=4.19803081186387E-16 -4.52415882534751E-15 -0.834690940757305
- joint arm_lower_top_plates_rotate: origin xyz=0.088000000461267 0.0462969388039673 -0.0518444185888435 rpy=3.14159265358973 1.37390099297363E-15 -3.14159265358979 -> xyz=0.0880000014350993 0.0462969374115836 -0.0518444513544338 rpy=3.14159265358973 -1.38777878078145E-17 -3.14159265358979
- joint arm_sync_plate_lower: origin xyz=0 0 0.0619999999999988 rpy=0.328597128236783 1.5707963267949 0 -> xyz=0 0 0.0619999994117862 rpy=0.328597211417039 1.5707963267949 0
- joint arm_sync_plates_rotate: origin xyz=0.534024004425634 0 -0.0659999999517558 rpy=0.0248080188130133 -1.57079631189374 -1.16632295052724 -> xyz=0.534023990063994 0 -0.0660000008575335 rpy=2.00092816921258 -1.5707963267949 0
- joint arm_top_actuator: axis -0.0879079473151551 0.996128602540272 0 -> -0.087908 0.99613 0; origin xyz=-0.0176725925011517 0.0587053523428329 0.0339996000000025 rpy=-8.6389229103645E-16 -1.1518563880486E-15 0.292409670050612 -> xyz=-0.017673 0.058705 0.034 rpy=-1.0547E-15 2.0262E-15 0.29241
- joint arm_top_actuator_rotate: origin xyz=-0.0898397083141685 -0.0340000000000132 0.333283716713238 rpy=1.5707963267949 -9.83199358550766E-16 -3.14159265358966 -> xyz=-0.089839708314947 -0.0339999999998062 0.333283716713238 rpy=1.5707963267949 2.49759149713076E-11 -3.14159265358966
- joint arm_top_actuator_top_rotate: origin xyz=-0.100495123315673 -0.178948287934891 -0.0419995999999991 rpy=-3.14159265358979 -5.48172618408671E-16 1.70371717647395 -> xyz=-0.100495120985836 -0.178948294411928 -0.0419995999999986 rpy=-3.14159265358979 -1.64451785522601E-15 1.70371714734334
- joint arm_top_plate_base_link: origin xyz=0 0 -0.0100000002511936 rpy=1.7589422877175 -1.5707963267949 0 -> xyz=0 0 -0.0100000028863516 rpy=1.75894227268368 -1.5707963267949 0
- joint back_left_leg_top_suspension: axis 0 0 -1 -> -1 0 0; origin xyz=0.0480999999999996 0.0906125308820751 0.00192206350156069 rpy=-1.5707963267949 0.208107268180907 1.5707963267949 -> xyz=0.00131825000000008 0.005 0.0199999999999999 rpy=3.14159265358979 7.08384070728071E-17 3.14159265358979
- joint back_left_swerve: type continuous -> fixed
- joint back_left_swerve_to_suspension: origin xyz=0.102203082302949 -0.0225748614789264 0.0671499999999996 rpy=-1.34 1.5707963267949 0 -> xyz=0.0203682500000001 0.190274606496618 0.0171061695141349 rpy=-5.01335084557297E-16 1.02633940524873E-16 3.14159265358979
- joint back_right_leg_base_joint: origin xyz=-0.27095694131393 -0.22418665200147 0.106000000000001 rpy=3.14159265358979 -1.22075621657598E-17 -7.14214183116779E-19 -> xyz=-0.27095694131393 -0.19918665200147 0.0860000000000012 rpy=-7.28583859910258E-17 2.77607356767723E-17 -3.14159265358979
- joint back_right_leg_top_suspension: axis 0 0 1 -> -1 0 0; origin xyz=-0.0480999999999999 0.0906125308820751 0.00192206350156076 rpy=1.5707963267949 0.208107268180907 1.5707963267949 -> xyz=-0.00131825000000008 0.03 0 rpy=0 -3.94348862876406E-34 0
- joint back_right_spring_joint: origin xyz=-0.01498 0.0379687078450422 0.0502559265692599 rpy=0 0.618421655113803 1.5707963267949 -> xyz=0.01498 0.0629687078450422 -0.0302559265692599 rpy=3.14159265358979 -0.618421655113803 1.5707963267949
- joint back_right_swerve: origin xyz=0.01905 0.01905 -0.166471215818396 rpy=6.88199027360824E-16 -1.24047364670461E-16 0.0539793695678587 -> xyz=0.0275730046201689 0.295196702840412 -0.271432246304261 rpy=-3.14159265358978 4.14560058185587E-17 -3.08761328402192; parent back_right_swerve_top -> back_right_leg_top; type continuous -> fixed
- joint back_right_wheel_axel: origin xyz=0 0.0640000971993742 -0.182000000000186 rpy=2.20205174609139 7.70217223333702E-16 1.57079632679491 -> xyz=0.0329052000000006 -0.186375097199374 0.0599328000001884 rpy=-0.939540907498405 -1.18689780226334E-14 -1.5707963267949
- joint claw_base: origin xyz=-0.437627718488799 -0.0353239921224943 0.021999999999998 rpy=1.5707963267949 -6.93889390390723E-17 -2.31503249752949 -> xyz=-0.437627735846881 -0.0353240159196297 0.0220000000000012 rpy=1.5707963267949 -5.68989300120393E-16 -2.3150326417559
- joint claw_left_close: axis 0 0.999999999999737 0 -> 0 0.999999999999955 0; origin xyz=-0.005930501944748 0.170021528163737 -0.0175355586756956 rpy=1.57079626487633 -1.13618506217272 5.38360649714105E-08 -> xyz=-0.00593050627315323 0.170021514327047 -0.017535510163561 rpy=1.57079678940594 -1.13618506217268 -4.02224433227641E-07
- joint claw_right_close: axis 0 -0.999999999999744 0 -> 0 -0.999999999999944 0; origin xyz=0.00593469734999167 0.170021528713698 0.017524087928418 rpy=-1.57079631288864 1.13618506217272 -3.14159264149837 -> xyz=0.00593469482197603 0.170021508317164 0.0175241162620443 rpy=-1.57079662358898 1.1361850621727 3.14159239553794
- joint claw_upper_link_joint: origin xyz=-0.00727246239987009 -0.0479999999999962 0.0230239566957189 rpy=1.07283329897131 1.70002900645727E-15 1.5707963267949 -> xyz=-0.00727258200204686 -0.0479999999999977 0.0230240155691104 rpy=1.07283343613791 2.12330153459561E-15 1.5707963267949
- joint claw_wrist_joint: axis 0 0.999999999998984 0 -> 0 0.999999999999683 0; origin xyz=-0.055634994248799 0 -0.0468700188956506 rpy=-4.03760624151054E-07 0.0889875109761181 -1.57079636267715 -> xyz=-0.0556350284488586 0 -0.0468700058001952 rpy=-1.25963063963236E-07 0.0889875109761248 -1.57079633798925
- joint front_left_back_to_rover_joint: mimic (none) -> joint=front_left_leg_top_suspension multiplier=1 offset=0
- joint front_left_leg_base_joint: origin xyz=0.271043058686069 0.22581334799853 0.106000000000001 rpy=-3.14159265358979 -7.45286116330806E-17 3.14159265358979 -> xyz=0.271043058686069 0.20081334799853 0.0860000000000011 rpy=1.38777878078144E-17 3.69020456027339E-18 -1.18444691579815E-31
- joint front_left_leg_top_suspension: axis 0 0 1 -> -1 0 0; origin xyz=-0.0481 0.0906125308820751 0.00192206350156074 rpy=1.5707963267949 0.208107268180907 1.5707963267949 -> xyz=-0.00131825000000006 0.03 0 rpy=0 3.01068278809724E-34 0
- joint front_left_spring_joint: origin xyz=0.01502 0.090421258375798 0.123974013894054 rpy=-1.5707963267949 0.618421655113804 1.5707963267949 -> xyz=-0.01502 0.115421258375798 -0.103974013894054 rpy=1.5707963267949 -0.618421655113804 1.5707963267949
- joint front_left_swerve: origin xyz=0.012974001894102 -0.0190500000000023 -0.144676938663704 rpy=1.51681695722705 1.48135988261336 -1.93089679672663E-15 -> xyz=0.0129740018941122 -0.0190499999998437 -0.144676938663703 rpy=1.51681695722842 1.48135988261336 -1.9308967967272E-15; type continuous -> fixed
- joint front_left_swerve_to_suspension: origin xyz=0.0875 0 0.06715 rpy=1.5707963267949 -6.479054612879E-16 0.297543712362438 -> xyz=-0.0177317499999999 0.171224606496618 0.0361561695141352 rpy=-1.90130020965652E-16 0.0894364441815313 1.5707963267949
- joint front_left_wheel_axel: origin xyz=0.222263715818585 -0.0640000971993724 0 rpy=-2.51033723429329 -2.85119150511548E-14 -1.5707963267949 -> xyz=0.222263715818585 -0.0640000971993911 0 rpy=-2.51033723429329 -1.39009637134535E-12 -1.5707963267949
- joint front_right_leg_base_joint: origin xyz=0.27104305868607 -0.22418665200147 0.106000000000001 rpy=3.14159265358979 -1.22075621657598E-17 -7.14214183116779E-19 -> xyz=0.27104 -0.19919 0.086 rpy=2.2031E-16 -4.6674E-17 -3.1416
- joint front_right_leg_top_suspension: axis 0 1 0 -> -1 0 0; origin xyz=-0.0349249999999999 0.005 0.02 rpy=3.14159265358979 0.208107268180909 1.5707963267949 -> xyz=-0.00131825000000007 0.03 0 rpy=0 -1.33808123915476E-34 0
- joint front_right_spring_joint: origin xyz=0.01502 0.090421258375798 0.123974013894054 rpy=-1.5707963267949 0.618421655113805 1.5707963267949 -> xyz=-0.01502 0.115421258375798 -0.103974013894054 rpy=1.5707963267949 -0.618421655113805 1.5707963267949
- joint front_right_swerve: origin xyz=0 -0.129521215818398 -0.0290322 rpy=-1.5707963267949 -1.51681695722704 0 -> xyz=0.00131825000000006 0.171224606496618 -0.149365046304261 rpy=-1.90254113716566E-16 -4.86879183181003E-17 -3.08761328402193; parent front_right_swerve_top -> front_right_leg_top; type continuous -> fixed
