Commit message: OWRS-204 #time 30m got the model loaded in gazebo, a few minor problems (see comments). Added in joint controllers for the drive, will have to do the same for swerve. Need to fix a few things in solidworks so it stands up. Hopefully should have it working tomorrow. Also had to make the suspension and arm joints fixed for now, so small steps to get everything working

File: rover/src/owr_bluetounge2_tf/robots/owr_bluetounge2_tf.URDF (robot description, URDF)
Before this commit: robot owr_bluetounge2_tf, 51 links, 50 joints
Links:
- link arm_bottom_actuator_base: mass 0.529218580973689 -> 0.529218581187352
- link arm_bottom_actuator_shaft: mass 0.834414953724233 -> 0.834414953724234
- link arm_bottom_plates: mass 0.523833534252721 -> 0.523833534252722
- link arm_top_actuator_base: mass 0.505108099842088 -> 0.50510809979627
- link arm_top_actuator_shaft: mass 0.707194769757717 -> 0.707194769757711
- link arm_top_plates: mass 0.632836443083173 -> 0.632836443083174
- link back_left_leg_top: mass 0.22831 -> 0.228308259818507
- link back_left_swerve_axel: mass 2.3439 -> 2.34386977405423
- link back_right_springs: mass 0.0728462856892432 -> 0.0728462856892431
- link base_link: mass 6.5755 -> 6.57554175926752
- link claw_base: mass 0.0771754639307836 -> 0.0771754639307835
- link claw_left: mass 0.0196972369456184 -> 0.0196972369456185
- link claw_wrist: mass 0.0918795943669827 -> 0.0918795943669828
- link front_left_swerve_axel: mass 2.36761790939096 -> 2.3676
- link front_right_leg_base: mass 0.085179 -> 0.0851788397766332
- link laser_tilt: mass 0.060913 -> 0.0609125923338383
Joints:
- joint arm_base_rotation: origin xyz=0.17255 -0.072487 0 rpy=5.7819E-16 -1.0312E-15 -0.088075 -> xyz=0.172554697757751 -0.0724869639786827 0 rpy=5.78193091528853E-16 -1.03121787249516E-15 -0.0880750381353883; type continuous -> fixed
- joint arm_bottom_actuator: limit lower=0 upper=0.31 effort=0 velocity=0 -> lower=0 upper=0.3 effort=0 velocity=0
- joint arm_bottom_actuator_base_rotate: limit effort=0 velocity=0 -> (none); origin xyz=0 0.088 -0.058 rpy=2.0009 -1.5708 0 -> xyz=0 0.0880000012352829 -0.0580000000598536 rpy=2.00092816923768 -1.5707963267949 0; type continuous -> fixed
- joint arm_bottom_plates_rotate: origin xyz=0.027518 -0.026 0.15313 rpy=1.5708 -1.1407 1.3825E-13 -> xyz=0.0275184819386707 -0.0259999999999941 0.153128001655061 rpy=1.57079632679489 -1.14066448437714 1.40494955389075E-13; type continuous -> fixed
- joint arm_lower_bottom_plates_rotate: origin xyz=-0.04722 0.44668 -0.022 rpy=-1.8388E-16 -3.3307E-16 -0.83469 -> xyz=-0.0472197994353847 0.446676986623695 -0.0219995999980227 rpy=4.19803081186387E-16 -4.52415882534751E-15 -0.834690940757305; type continuous -> fixed
- joint arm_lower_top_plates_rotate: origin xyz=0.088 0.046297 -0.051844 rpy=3.1416 -1.3878E-17 -3.1416 -> xyz=0.0880000014350993 0.0462969374115836 -0.0518444513544338 rpy=3.14159265358973 -1.38777878078145E-17 -3.14159265358979; type continuous -> fixed
- joint arm_sync_plate_lower: origin xyz=0 0 0.062 rpy=0.3286 1.5708 0 -> xyz=0 0 0.0619999994117862 rpy=0.328597211417039 1.5707963267949 0; type continuous -> fixed
- joint arm_sync_plates_rotate: origin xyz=0.53402 0 -0.066 rpy=2.0009 -1.5708 0 -> xyz=0.534023990063994 0 -0.0660000008575335 rpy=2.00092816921258 -1.5707963267949 0; type continuous -> fixed
- joint arm_top_actuator: limit lower=0 upper=0.26 effort=0 velocity=0 -> lower=0 upper=0.3 effort=0 velocity=0; origin xyz=-0.017673 0.058705 0.034 rpy=-8.9165E-16 -1.3323E-15 0.29241 -> xyz=-0.017673 0.058705 0.034 rpy=-1.0547E-15 2.0262E-15 0.29241
- joint arm_top_actuator_rotate: origin xyz=-0.08984 -0.034 0.33328 rpy=1.5708 2.4976E-11 -3.1416 -> xyz=-0.089839708314947 -0.0339999999998062 0.333283716713238 rpy=1.5707963267949 2.49759149713076E-11 -3.14159265358966; type continuous -> fixed
- joint arm_top_actuator_top_rotate: limit effort=0 velocity=0 -> (none); origin xyz=-0.1005 -0.17895 -0.042 rpy=-3.1416 -4.2327E-16 1.7037 -> xyz=-0.100495120985836 -0.178948294411928 -0.0419995999999986 rpy=-3.14159265358979 -1.64451785522601E-15 1.70371714734334; type continuous -> fixed
- joint arm_top_plate_base_link: origin xyz=0 0 -0.01 rpy=1.7589 -1.5708 0 -> xyz=0 0 -0.0100000028863516 rpy=1.75894227268368 -1.5707963267949 0; type continuous -> fixed
- joint back_left_leg_base_joint: origin xyz=-0.27096 0.22581 0.106 rpy=3.1416 -7.4529E-17 3.1416 -> xyz=-0.27095694131393 0.22581334799853 0.106000000000001 rpy=3.14159265358979 -7.45286116330805E-17 3.14159265358979
- joint back_left_leg_top_suspension: origin xyz=0.0013183 0.005 0.02 rpy=3.1416 7.0838E-17 3.1416 -> xyz=0.00131825000000008 0.005 0.0199999999999999 rpy=3.14159265358979 7.08384070728071E-17 3.14159265358979; type continuous -> fixed
- joint back_left_spring_joint: origin xyz=0.01502 0.037969 0.050256 rpy=-1.0645E-16 0.61842 1.5708 -> xyz=0.01502 0.0379687078450422 0.0502559265692599 rpy=-1.06451592460411E-16 0.618421655113802 1.5707963267949
- joint back_left_suspension_joint: axis 0 0 -1 -> 0 0 1; origin xyz=0 0.015 0.09615 rpy=1.5708 -0.85597 3.1416 -> xyz=0 0.0149999999999999 0.09615 rpy=1.5707963267949 -0.855968458217554 3.14159265358979; type continuous -> fixed
- joint back_left_swerve: type continuous -> fixed
- joint back_left_swerve_to_suspension: origin xyz=0.020368 0.19027 0.017106 rpy=-5.0134E-16 1.0263E-16 3.1416 -> xyz=0.0203682500000001 0.190274606496618 0.0171061695141349 rpy=-5.01335084557297E-16 1.02633940524873E-16 3.14159265358979; type continuous -> fixed
- joint back_left_to_rover_joint: origin xyz=-0.0072603 -0.097363 2E-05 rpy=0.096406 1.5708 0 -> xyz=-0.0072603045458083 -0.0973626127237505 2.00000000003531E-05 rpy=0.0964062134635395 1.5707963267949 0; type continuous -> fixed
- joint back_left_wheel_axel: origin xyz=0 0.064 -0.182 rpy=2.2021 7.7022E-16 1.5708 -> xyz=0 0.0640000971993742 -0.182000000000186 rpy=2.20205174609139 7.70217223333702E-16 1.57079632679491
- joint back_right_leg_base_joint: origin xyz=-0.27096 -0.19919 0.086 rpy=-7.2858E-17 2.7761E-17 -3.1416 -> xyz=-0.27095694131393 -0.19918665200147 0.0860000000000012 rpy=-7.28583859910258E-17 2.77607356767723E-17 -3.14159265358979
- joint back_right_leg_top_suspension: origin xyz=-0.0013183 0.03 0 rpy=0 -3.9435E-34 0 -> xyz=-0.00131825000000008 0.03 0 rpy=0 -3.94348862876406E-34 0; type continuous -> fixed
- joint back_right_spring_joint: origin xyz=0.01498 0.062969 -0.030256 rpy=3.1416 -0.61842 1.5708 -> xyz=0.01498 0.0629687078450422 -0.0302559265692599 rpy=3.14159265358979 -0.618421655113803 1.5707963267949
- joint back_right_suspension_joint: origin xyz=0.0059835 0.03312 0.082395 rpy=1.5708 -0.41031 0 -> xyz=0.00598346458625637 0.03312 0.082395068101082 rpy=1.5707963267949 -0.410314386932896 0; type continuous -> fixed
- joint back_right_swerve: origin xyz=0.027573 0.2952 -0.27143 rpy=-3.1416 4.1456E-17 -3.0876 -> xyz=0.0275730046201689 0.295196702840412 -0.271432246304261 rpy=-3.14159265358978 4.14560058185587E-17 -3.08761328402192; type continuous -> fixed
- joint back_right_to_rover_joint: origin xyz=-0.090706 -0.021118 0.0481 rpy=1.7789 -1.5708 0 -> xyz=-0.090706394544977 -0.0211184214377016 0.0480999999999998 rpy=1.7789035949758 -1.5707963267949 0; type continuous -> fixed
- joint back_right_wheel_axel: origin xyz=0.032905 -0.18638 0.059933 rpy=-0.93954 -1.1869E-14 -1.5708 -> xyz=0.0329052000000006 -0.186375097199374 0.0599328000001884 rpy=-0.939540907498405 -1.18689780226334E-14 -1.5707963267949
- joint claw_base: origin xyz=-0.43763 -0.035324 0.022 rpy=1.5708 -2.6368E-16 -2.315 -> xyz=-0.437627735846881 -0.0353240159196297 0.0220000000000012 rpy=1.5707963267949 -5.68989300120393E-16 -2.3150326417559; type continuous -> fixed
- joint claw_left_close: axis 0 1 0 -> 0 0.999999999999955 0; origin xyz=-0.0059305 0.17002 -0.017536 rpy=1.5708 -1.1362 -1.338E-07 -> xyz=-0.00593050627315323 0.170021514327047 -0.017535510163561 rpy=1.57079678940594 -1.13618506217268 -4.02224433227641E-07; type continuous -> fixed
- joint claw_right_close: axis 0 -1 0 -> 0 -0.999999999999944 0; origin xyz=0.0059347 0.17002 0.017524 rpy=-1.5708 1.1362 3.1416 -> xyz=0.00593469482197603 0.170021508317164 0.0175241162620443 rpy=-1.57079662358898 1.1361850621727 3.14159239553794; type continuous -> fixed
- joint claw_upper_link_joint: origin xyz=-0.0072725 -0.048 0.023024 rpy=1.0728 2.3453E-15 1.5708 -> xyz=-0.00727258200204686 -0.0479999999999977 0.0230240155691104 rpy=1.07283343613791 2.12330153459561E-15 1.5707963267949; type continuous -> fixed
- joint claw_wrist_joint: axis 0 1 0 -> 0 0.999999999999683 0; origin xyz=-0.055635 0 -0.04687 rpy=-5.5546E-09 0.088988 -1.5708 -> xyz=-0.0556350284488586 0 -0.0468700058001952 rpy=-1.25963063963236E-07 0.0889875109761248 -1.57079633798925; type continuous -> fixed
- joint front_left_back_to_rover_joint: mimic (none) -> joint=front_left_leg_top_suspension multiplier=1 offset=0; origin xyz=-0.090706 0.021118 0.0481 rpy=1.7789 1.5708 0 -> xyz=-0.0907063945449771 0.0211184214377016 0.0481 rpy=1.7789035949758 1.5707963267949 0; type continuous -> fixed
- joint front_left_leg_base_joint: origin xyz=0.27104 0.20081 0.086 rpy=1.3878E-17 3.6902E-18 -1.1844E-31 -> xyz=0.271043058686069 0.20081334799853 0.0860000000000011 rpy=1.38777878078144E-17 3.69020456027339E-18 -1.18444691579815E-31
- joint front_left_leg_top_suspension: origin xyz=-0.0013183 0.03 0 rpy=0 3.0107E-34 0 -> xyz=-0.00131825000000006 0.03 0 rpy=0 3.01068278809724E-34 0; type continuous -> fixed
- joint front_left_spring_joint: origin xyz=-0.01502 0.11542 -0.10397 rpy=1.5708 -0.61842 1.5708 -> xyz=-0.01502 0.115421258375798 -0.103974013894054 rpy=1.5707963267949 -0.618421655113804 1.5707963267949
- joint front_left_suspension_joint: origin xyz=0.0059835 0.0080794 -0.03308 rpy=0 0 -0.41031 -> xyz=0.00598346458625643 0.00807938385087792 -0.0330799999999998 rpy=0 0 -0.410314386932897; type continuous -> fixed
- joint front_left_swerve: origin xyz=0.012974 -0.01905 -0.14468 rpy=1.5168 1.4814 -1.9309E-15 -> xyz=0.0129740018941122 -0.0190499999998437 -0.144676938663703 rpy=1.51681695722842 1.48135988261336 -1.9308967967272E-15; type continuous -> fixed
- joint front_left_swerve_to_suspension: origin xyz=-0.017732 0.17122 0.036156 rpy=-1.9013E-16 0.089436 1.5708 -> xyz=-0.0177317499999999 0.171224606496618 0.0361561695141352 rpy=-1.90130020965652E-16 0.0894364441815313 1.5707963267949; type continuous -> fixed
- joint front_left_wheel_axel: origin xyz=0.22226 -0.064 0 rpy=-2.5103 -1.3901E-12 -1.5708 -> xyz=0.222263715818585 -0.0640000971993911 0 rpy=-2.51033723429329 -1.39009637134535E-12 -1.5707963267949
- joint front_right_leg_top_suspension: origin xyz=-0.0013183 0.03 0 rpy=0 -1.3381E-34 0 -> xyz=-0.00131825000000007 0.03 0 rpy=0 -1.33808123915476E-34 0; type continuous -> fixed
- joint front_right_spring_joint: origin xyz=-0.01502 0.11542 -0.10397 rpy=1.5708 -0.61842 1.5708 -> xyz=-0.01502 0.115421258375798 -0.103974013894054 rpy=1.5707963267949 -0.618421655113805 1.5707963267949
- joint front_right_suspension_joint: origin xyz=0.0059835 0.0080794 -0.03308 rpy=0 -3.4694E-16 -0.41031 -> xyz=0.00598346458625632 0.00807938385087792 -0.0330799999999998 rpy=0 -3.46944695195361E-16 -0.410314386932897; type continuous -> fixed
- joint front_right_swerve: origin xyz=0.0013183 0.17122 -0.14937 rpy=-1.9025E-16 -4.8688E-17 -3.0876 -> xyz=0.00131825000000006 0.171224606496618 -0.149365046304261 rpy=-1.90254113716566E-16 -4.86879183181003E-17 -3.08761328402193; type continuous -> fixed
- joint front_right_to_rover_joint: origin xyz=-0.090706 0.021118 0.0481 rpy=1.7789 1.5708 0 -> xyz=-0.0907063945449771 0.0211184214377016 0.0481000000000001 rpy=1.7789035949758 1.5707963267949 0; type continuous -> fixed
- joint front_right_wheel_axel: origin xyz=0 0.064 -0.182 rpy=2.2021 1.9325E-15 1.5708 -> xyz=0 0.0640000971993744 -0.182000000000186 rpy=2.20205174609138 1.93248195223816E-15 1.57079632679491
- joint laser_tilt_base: origin xyz=0.26214 0.16581 0.116 rpy=-4.0766E-16 -2.7114E-15 -7.1421E-19 -> xyz=0.26213671627839 0.165813347998531 0.116 rpy=-4.0766001685455E-16 -2.71143453751384E-15 -7.14214183115679E-19
- joint laser_tilt_joint: limit lower=-1.5708 upper=0.785298 effort=0 velocity=0 -> lower=-0.785398 upper=1.5708 effort=0 velocity=0; origin xyz=-0.0069285 -0.01905 0.029 rpy=-1.5708 1.0852 0 -> xyz=-0.00692854336717914 -0.01905 0.029 rpy=-1.5707963267949 1.08521967863993 0
- joint lidar_frame_base: origin xyz=-0.092214 -0.039413 0.034656 rpy=1.5708 0.11022 -1.0852 -> xyz=-0.0922144508966998 -0.0394134633802184 0.0346559749585283 rpy=1.5707963267949 0.110221873047514 -1.08521967863993

Commit message: OWRS-204 #time 30m a few fixes

File: rover/src/owr_bluetounge2_tf/robots/owr_bluetounge2_tf.URDF (robot description, URDF)
Before this commit: robot owr_bluetounge2_tf, 53 links, 52 joints
Links:
- added link chassis, mass 6.57554175926752; collision mesh filename=package://owr_bluetounge2_tf/meshes/base_link.STL; visual mesh filename=package://owr_bluetounge2_tf/meshes/base_link.STL
- link base_link: mass 6.57554175926752 -> None; geometry 
Joints:
- added joint base_link_joint: type fixed, parent base_link, child chassis, origin xyz=0 0 0  rpy=0 0 0, axis 0 0 0
- joint arm_base_rotation: parent base_link -> chassis
- joint back_left_leg_base_joint: parent base_link -> chassis
- joint back_right_leg_base_joint: parent base_link -> chassis
- joint front_left_leg_base_joint: parent base_link -> chassis
- joint front_right_leg_base_joint: parent base_link -> chassis
- joint laser_tilt_base: parent base_link -> chassis

Commit message: OWRS-204 forgot to commit this, not sure how long was spent

File: rover/src/owr_bluetounge2_tf/robots/owr_bluetounge2_tf.URDF (robot description, URDF)
Before this commit: robot owr_bluetounge2_tf, 53 links, 52 joints
Joints:
- joint back_right_swerve_to_suspension: axis 0 0 0 -> -1 0 0; type fixed -> continuous

Commit message: OWRS-204 #time 30m fixed the urdf so it is now working

File: rover/src/owr_bluetounge2_tf/robots/owr_bluetounge2_tf.URDF (robot description, URDF)
Before this commit: robot owr_bluetounge2_tf, 54 links, 53 joints
Joints:
- joint back_right_swerve_to_suspension: origin xyz=0.102203082302949 0.0225748614789264 0.0290499999999999 rpy=1.36268905861399 -1.5707963267949 0 -> xyz=0.102203082302949 0.0225748614789264 0.0290499999999999 rpy=1.72268905861399 -1.5707963267949 0; type continuous -> fixed

Commit message: OWRS-203 #time 20m some bug fixes for drive motors

File: rover/src/owr_bluetounge2_tf/robots/owr_bluetounge2_tf.URDF (robot description, URDF)
Before this commit: robot owr_bluetounge2_tf, 54 links, 53 joints
Joints:
- joint front_left_swerve: axis -1 0 0 -> 1 0 0

Commit message: OWRS-175 #time 10m created static transform for slam in urdf whilst lidar is not working

File: rover/src/owr_bluetounge2_tf/robots/owr_bluetounge2_tf.URDF (robot description, URDF)
Before this commit: robot owr_bluetounge2_tf, 54 links, 53 joints
Links:
- added link base_stabalized_frame
Joints:
- added joint base_footprint_joint: type fixed, parent base_footprint, child base_link, origin xyz=0 0 0  rpy=0 0 0, axis 0 0 0

Commit message: OWRS-175 #time 30m slam setup correctly and all tfs working

File: rover/src/owr_bluetounge2_tf/robots/owr_bluetounge2_tf.URDF (robot description, URDF)
Before this commit: robot owr_bluetounge2_tf, 55 links, 54 joints
Links:
- removed link base_stabalized_frame
- added link base_footprint

Commit message: OWRS-237 #time 15m design and updating the simulator to support arm rotation

File: rover/src/owr_bluetounge2_tf/robots/owr_bluetounge2_tf.URDF (robot description, URDF)
Before this commit: robot owr_bluetounge2_tf, 55 links, 54 joints
Joints:
- joint arm_base_rotation: type fixed -> continuous

Commit message: OWRS-278 #time 4h seems to fuse okish

File: rover/src/owr_bluetounge2_tf/robots/owr_bluetounge2_tf.URDF (robot description, URDF)
Before this commit: robot owr_bluetounge2_tf, 55 links, 54 joints
Links:
- added link clinometer
Joints:
- added joint clinometer_joint: type fixed, parent base_link, child clinometer, origin xyz=0 0 0 rpy=0 0 3.14159, axis 0 0 0

Commit message: OWRS-175 #time 3h Different localisation options for tomorrow

File: rover/src/owr_bluetounge2_tf/robots/owr_bluetounge2_tf.URDF (robot description, URDF)
Before this commit: robot owr_bluetounge2_tf, 56 links, 55 joints
Joints:
- joint base_footprint_joint: origin xyz=0 0 0  rpy=0 0 0 -> xyz=0 0 .3  rpy=0 0 0
