Commit message: Fixed package info

File: rover/src/owr_numbat_tf/urdf/Assembly.SLDASM.urdf (robot description, URDF)
Before this commit: robot Assembly.SLDASM, 9 links, 8 joints
Links:
- link Back Left Axle: geometry collision mesh filename=package://owr_numbat_tf/meshes/Back Left Axle.STL; visual mesh filename=package://owr_numbat_tf/meshes/Back Left Axle.STL
- link Back Left Wheel: geometry collision mesh filename=package://owr_numbat_tf/meshes/Back Left Wheel.STL; visual mesh filename=package://owr_numbat_tf/meshes/Back Left Wheel.STL
- link Back Right Axle: geometry collision mesh filename=package://owr_numbat_tf/meshes/Back Right Axle.STL; visual mesh filename=package://owr_numbat_tf/meshes/Back Right Axle.STL
- link Back Right Wheel: geometry collision mesh filename=package://owr_numbat_tf/meshes/Back Right Wheel.STL; visual mesh filename=package://owr_numbat_tf/meshes/Back Right Wheel.STL
- link Front Left Axle: geometry collision mesh filename=package://owr_numbat_tf/meshes/Front Left Axle.STL; visual mesh filename=package://owr_numbat_tf/meshes/Front Left Axle.STL
- link Front Left wheel: geometry collision mesh filename=package://owr_numbat_tf/meshes/Front Left wheel.STL; visual mesh filename=package://owr_numbat_tf/meshes/Front Left wheel.STL
- link Front RIght Wheel: geometry collision mesh filename=package://owr_numbat_tf/meshes/Front RIght Wheel.STL; visual mesh filename=package://owr_numbat_tf/meshes/Front RIght Wheel.STL
- link Front Right Axle: geometry collision mesh filename=package://owr_numbat_tf/meshes/Front Right Axle.STL; visual mesh filename=package://owr_numbat_tf/meshes/Front Right Axle.STL
- link base_link: geometry collision mesh filename=package://owr_numbat_tf/meshes/base_link.STL; visual mesh filename=package://owr_numbat_tf/meshes/base_link.STL
