Commit message: Added laser tilt to urdf

File: rover/src/owr_numbat_tf/robots/owr_numbat_tf.urdf (robot description, URDF)
Before this commit: robot owr_numbat_tf, 9 links, 8 joints
Links:
- added link laser_tilt, mass 0.0609125923338383; collision mesh filename=package://owr_bluetounge2_tf/meshes/laser_tilt.STL; visual mesh filename=package://owr_bluetounge2_tf/meshes/laser_tilt.STL
- added link laser_tilt_tilt, mass 0.063245803268312; collision mesh filename=package://owr_bluetounge2_tf/meshes/laser_tilt_tilt.STL; visual mesh filename=package://owr_bluetounge2_tf/meshes/laser_tilt_tilt.STL
- added link lidar_frame, mass 0.229160254803044; collision mesh filename=package://owr_bluetounge2_tf/meshes/lidar_frame.STL; visual mesh filename=package://owr_bluetounge2_tf/meshes/lidar_frame.STL
Joints:
- added joint laser_tilt_base: type fixed, parent base_link, child laser_tilt, origin xyz=0.26213671627839 0.165813347998531 0.116 rpy=-4.0766001685455E-16 -2.71143453751384E-15 -7.14214183115679E-19, axis 0 0 0
- added joint laser_tilt_joint: type revolute, parent laser_tilt, child laser_tilt_tilt, origin xyz=-0.00692854336717914 -0.01905 0.029 rpy=-1.5707963267949 1.08521967863993 0, axis 0 0 1, limit lower=-0.785398 upper=1.5708 effort=0 velocity=0
- added joint lidar_frame_base: type fixed, parent laser_tilt_tilt, child lidar_frame, origin xyz=-0.0922144508966998 -0.0394134633802184 0.0346559749585283 rpy=1.5707963267949 0.110221873047514 -1.08521967863993, axis 0 0 0

Commit message: Placed lidar and gimbal in correct position

File: rover/src/owr_numbat_tf/robots/owr_numbat_tf.urdf (robot description, URDF)
Before this commit: robot owr_numbat_tf, 12 links, 11 joints
Joints:
- joint laser_tilt_base: origin xyz=0.26213671627839 0.165813347998531 0.116 rpy=-4.0766001685455E-16 -2.71143453751384E-15 -7.14214183115679E-19 -> xyz=0.5 -0.75 0.47 rpy=-4.0766001685455E-16 -2.71143453751384E-15 -7.14214183115679E-19

Commit message: Fixed joint names so they are in the right directiony

File: rover/src/owr_numbat_tf/robots/owr_numbat_tf.urdf (robot description, URDF)
Before this commit: robot owr_numbat_tf, 12 links, 11 joints
Links:
- removed link Back Left Axle
- removed link Back Left Wheel
- removed link Back Right Axle
- removed link Back Right Wheel
- removed link Front Left Axle
- removed link Front Left wheel
- removed link Front Right Axle
- added link back_left Axle, mass 0.674113164049983; collision mesh filename=package://owr_numbat_tf/meshes/Front Right Axle.STL; visual mesh filename=package://owr_numbat_tf/meshes/Front Right Axle.STL
- added link back_right Axle, mass 0.674113164049984; collision mesh filename=package://owr_numbat_tf/meshes/Front Left Axle.STL; visual mesh filename=package://owr_numbat_tf/meshes/Front Left Axle.STL
- added link back_right wheel, mass 1.5442893046468; collision mesh filename=package://owr_numbat_tf/meshes/Front Left wheel.STL; visual mesh filename=package://owr_numbat_tf/meshes/Front Left wheel.STL
- added link front_left Axle, mass 0.674113164049983; collision mesh filename=package://owr_numbat_tf/meshes/Back Right Axle.STL; visual mesh filename=package://owr_numbat_tf/meshes/Back Right Axle.STL
- added link front_left Wheel, mass 1.54428930464679; collision mesh filename=package://owr_numbat_tf/meshes/Back Right Wheel.STL; visual mesh filename=package://owr_numbat_tf/meshes/Back Right Wheel.STL
- added link front_right Axle, mass 0.674113164049983; collision mesh filename=package://owr_numbat_tf/meshes/Back Left Axle.STL; visual mesh filename=package://owr_numbat_tf/meshes/Back Left Axle.STL
- added link front_right Wheel, mass 1.5442893046468; collision mesh filename=package://owr_numbat_tf/meshes/Back Left Wheel.STL; visual mesh filename=package://owr_numbat_tf/meshes/Back Left Wheel.STL
Joints:
- removed joint Back Left Rotate
- removed joint Back Left Steer
- removed joint Back Right Steer
- removed joint Front Left Steer
- removed joint Front Left rotate
- removed joint Front Right Rotate
- removed joint Front Right Steer
- added joint back_left Rotate: type continuous, parent back_left Axle, child Front RIght Wheel, origin xyz=0 0.0299999999999999 0 rpy=-1.5707963267949 -0.00858284690216311 1.57079632679489, axis 0 0 1
- added joint back_left Steer: type continuous, parent base_link, child back_left Axle, origin xyz=0.626839262679528 -0.884494656994069 0.13494946923044 rpy=1.5707963267949 6.12114355045412E-17 1.54596104769157, axis 0 1 0
- added joint back_right Steer: type continuous, parent base_link, child back_right Axle, origin xyz=0.62684 -0.40335 0.13495 rpy=1.5708 6.088E-17 1.6778, axis 0 1 0
- added joint back_right rotate: type continuous, parent back_right Axle, child back_right wheel, origin xyz=0 0.03 0 rpy=-1.5708 -0.91526 1.5708, axis 0 0 1
- added joint front_left Steer: type continuous, parent base_link, child front_left Axle, origin xyz=-0.13031 -0.88449 0.13495 rpy=1.5708 5.9043E-17 1.3027, axis 0 1 0
- added joint front_right Rotate: type continuous, parent front_right Axle, child front_right Wheel, origin xyz=0 0.0300000000000001 0 rpy=1.57079632679489 0.214040970418392 -1.5707963267949, axis 0 0 1
- added joint front_right Steer: type continuous, parent base_link, child front_right Axle, origin xyz=-0.13031 -0.40335 0.13495 rpy=1.5708 6.0901E-17 1.4671, axis 0 1 0
- joint Back RIght Rotate: child Back Right Wheel -> front_left Wheel; parent Back Right Axle -> front_left Axle
- joint laser_tilt_base: origin xyz=0.5 -0.75 0.47 rpy=-4.0766001685455E-16 -2.71143453751384E-15 -7.14214183115679E-19 -> xyz=-0.1 -0.75 0.47 rpy=-4.0766001685455E-16 2.71143453751384E-15 -3.14214183115679

Commit message: Added base_link to subsitution rover

File: rover/src/owr_numbat_tf/robots/owr_numbat_tf.urdf (robot description, URDF)
Before this commit: robot owr_numbat_tf, 12 links, 11 joints
Links:
- added link rover_model, mass 33.4975943636999; collision mesh filename=package://owr_numbat_tf/meshes/rover_model.STL; visual mesh filename=package://owr_numbat_tf/meshes/rover_model.STL
- link base_link: mass 33.4975943636999 -> None; geometry 
Joints:
- added joint base_link_rover: type fixed, parent base_link, child rover_model, origin xyz=-0.1 -0.6 0 rpy=0 0 0, axis 0 0 0
- joint back_left Steer: parent base_link -> rover_model
- joint back_right Steer: parent base_link -> rover_model
- joint front_left Steer: parent base_link -> rover_model
- joint front_right Steer: parent base_link -> rover_model
- joint laser_tilt_base: parent base_link -> rover_model

Commit message: Fix stl reference

File: rover/src/owr_numbat_tf/robots/owr_numbat_tf.urdf (robot description, URDF)
Before this commit: robot owr_numbat_tf, 13 links, 12 joints
Links:
- link rover_model: geometry collision mesh filename=package://owr_numbat_tf/meshes/base_link.STL; visual mesh filename=package://owr_numbat_tf/meshes/base_link.STL

Commit message: Renamed joints to match bluetongue

File: rover/src/owr_numbat_tf/robots/owr_numbat_tf.urdf (robot description, URDF)
Before this commit: robot owr_numbat_tf, 13 links, 12 joints
Joints:
- removed joint back_left Steer
- removed joint back_right Steer
- removed joint front_left Steer
- removed joint front_right Steer
- added joint back_left_swerve: type continuous, parent rover_model, child back_left Axle, origin xyz=0.626839262679528 -0.884494656994069 0.13494946923044 rpy=1.5707963267949 6.12114355045412E-17 1.54596104769157, axis 0 1 0
- added joint back_right_swerve: type continuous, parent rover_model, child back_right Axle, origin xyz=0.62684 -0.40335 0.13495 rpy=1.5708 6.088E-17 1.6778, axis 0 1 0
- added joint front_left_swerve: type continuous, parent rover_model, child front_left Axle, origin xyz=-0.13031 -0.88449 0.13495 rpy=1.5708 5.9043E-17 1.3027, axis 0 1 0
- added joint front_right_swerve: type continuous, parent rover_model, child front_right Axle, origin xyz=-0.13031 -0.40335 0.13495 rpy=1.5708 6.0901E-17 1.4671, axis 0 1 0
- joint base_link_rover: origin xyz=-0.1 -0.6 0 rpy=0 0 0 -> xyz=0.2 -0.65 0 rpy=0 0 3.14159265359

Commit message: Fixed finally joint naming mistakes in urdf

File: rover/src/owr_numbat_tf/robots/owr_numbat_tf.urdf (robot description, URDF)
Before this commit: robot owr_numbat_tf, 13 links, 12 joints
Links:
- removed link back_left Axle
- removed link back_right Axle
- removed link front_left Axle
- removed link front_right Axle
- added link back_left_wheel_axel, mass 0.674113164049983; collision mesh filename=package://owr_numbat_tf/meshes/Front Right_wheel_axel.STL; visual mesh filename=package://owr_numbat_tf/meshes/Front Right_wheel_axel.STL
- added link back_right_wheel_axel, mass 0.674113164049984; collision mesh filename=package://owr_numbat_tf/meshes/Front Left_wheel_axel.STL; visual mesh filename=package://owr_numbat_tf/meshes/Front Left_wheel_axel.STL
- added link front_left_wheel_axel, mass 0.674113164049983; collision mesh filename=package://owr_numbat_tf/meshes/Back Right_wheel_axel.STL; visual mesh filename=package://owr_numbat_tf/meshes/Back Right_wheel_axel.STL
- added link front_right_wheel_axel, mass 0.674113164049983; collision mesh filename=package://owr_numbat_tf/meshes/Back Left_wheel_axel.STL; visual mesh filename=package://owr_numbat_tf/meshes/Back Left_wheel_axel.STL
- link laser_tilt: geometry collision mesh filename=package://owr_numbat_tf/meshes/laser_tilt.STL; visual mesh filename=package://owr_numbat_tf/meshes/laser_tilt.STL
- link laser_tilt_tilt: geometry collision mesh filename=package://owr_numbat_tf/meshes/laser_tilt_tilt.STL; visual mesh filename=package://owr_numbat_tf/meshes/laser_tilt_tilt.STL
- link lidar_frame: geometry collision mesh filename=package://owr_numbat_tf/meshes/lidar_frame.STL; visual mesh filename=package://owr_numbat_tf/meshes/lidar_frame.STL
Joints:
- removed joint Back RIght Rotate
- removed joint back_left Rotate
- removed joint front_right Rotate
- added joint Back RIght_wheel_axel: type continuous, parent front_left_wheel_axel, child front_left Wheel, origin xyz=0 0.0299999999999999 0 rpy=-1.57079632679491 -1.13219561486008 1.57079632679491, axis 0 0 1
- added joint back_left_wheel_axel: type continuous, parent back_left_wheel_axel, child Front RIght Wheel, origin xyz=0 0.0299999999999999 0 rpy=-1.5707963267949 -0.00858284690216311 1.57079632679489, axis 0 0 1
- added joint front_right_wheel_axel: type continuous, parent front_right_wheel_axel, child front_right Wheel, origin xyz=0 0.0300000000000001 0 rpy=1.57079632679489 0.214040970418392 -1.5707963267949, axis 0 0 1
- joint back_left_swerve: child back_left Axle -> back_left_wheel_axel
- joint back_right rotate: parent back_right Axle -> back_right_wheel_axel
- joint back_right_swerve: child back_right Axle -> back_right_wheel_axel
- joint front_left_swerve: child front_left Axle -> front_left_wheel_axel
- joint front_right_swerve: child front_right Axle -> front_right_wheel_axel

Commit message: Fix stl name

File: rover/src/owr_numbat_tf/robots/owr_numbat_tf.urdf (robot description, URDF)
Before this commit: robot owr_numbat_tf, 13 links, 12 joints
Links:
- link back_left_wheel_axel: geometry collision mesh filename=package://owr_numbat_tf/meshes/Front Right Axel.STL; visual mesh filename=package://owr_numbat_tf/meshes/Front Right Axel.STL
- link back_right_wheel_axel: geometry collision mesh filename=package://owr_numbat_tf/meshes/Front Left Axel.STL; visual mesh filename=package://owr_numbat_tf/meshes/Front Left Axel.STL
- link front_left_wheel_axel: geometry collision mesh filename=package://owr_numbat_tf/meshes/Back Right Axel.STL; visual mesh filename=package://owr_numbat_tf/meshes/Back Right Axel.STL
- link front_right_wheel_axel: geometry collision mesh filename=package://owr_numbat_tf/meshes/Back Left Axel.STL; visual mesh filename=package://owr_numbat_tf/meshes/Back Left Axel.STL

Commit message: Fix stl name

File: rover/src/owr_numbat_tf/robots/owr_numbat_tf.urdf (robot description, URDF)
Before this commit: robot owr_numbat_tf, 13 links, 12 joints
Links:
- link back_left_wheel_axel: geometry collision mesh filename=package://owr_numbat_tf/meshes/Front Right Axle.STL; visual mesh filename=package://owr_numbat_tf/meshes/Front Right Axle.STL
- link back_right_wheel_axel: geometry collision mesh filename=package://owr_numbat_tf/meshes/Front Left Axle.STL; visual mesh filename=package://owr_numbat_tf/meshes/Front Left Axle.STL
- link front_left_wheel_axel: geometry collision mesh filename=package://owr_numbat_tf/meshes/Back Right Axle.STL; visual mesh filename=package://owr_numbat_tf/meshes/Back Right Axle.STL
- link front_right_wheel_axel: geometry collision mesh filename=package://owr_numbat_tf/meshes/Back Left Axle.STL; visual mesh filename=package://owr_numbat_tf/meshes/Back Left Axle.STL
Joints:
- removed joint Back RIght_wheel_axel
- added joint back_right_wheel_axel: type continuous, parent front_left_wheel_axel, child front_left Wheel, origin xyz=0 0.0299999999999999 0 rpy=-1.57079632679491 -1.13219561486008 1.57079632679491, axis 0 0 1

Commit message: Urdf correct

File: rover/src/owr_numbat_tf/robots/owr_numbat_tf.urdf (robot description, URDF)
Before this commit: robot owr_numbat_tf, 13 links, 12 joints
Joints:
- removed joint back_right rotate
- added joint front_left_wheel_axel: type continuous, parent front_left_wheel_axel, child front_left Wheel, origin xyz=0 0.0299999999999999 0 rpy=-1.57079632679491 -1.13219561486008 1.57079632679491, axis 0 0 1
- joint back_right_wheel_axel: child front_left Wheel -> back_right wheel; origin xyz=0 0.0299999999999999 0 rpy=-1.57079632679491 -1.13219561486008 1.57079632679491 -> xyz=0 0.03 0 rpy=-1.5708 -0.91526 1.5708; parent front_left_wheel_axel -> back_right_wheel_axel

Commit message: Code comments and cleanups

File: rover/src/owr_numbat_tf/robots/owr_numbat_tf.urdf (robot description, URDF)
Before this commit: robot owr_numbat_tf, 13 links, 12 joints
Links:
- removed link Front RIght Wheel
- added link front_right_Wheel, mass 1.54428930379881; collision mesh filename=package://owr_numbat_tf/meshes/Front RIght Wheel.STL; visual mesh filename=package://owr_numbat_tf/meshes/Front RIght Wheel.STL
Joints:
- removed joint back_right rotate
- added joint front_left_wheel_axel: type continuous, parent back_left_wheel_axel, child front_right_Wheel, origin xyz=0 0.0299999999999999 0 rpy=-1.5707963267949 -0.00858284690216311 1.57079632679489, axis 0 0 1
- joint back_left_wheel_axel: child Front RIght Wheel -> back_right wheel; origin xyz=0 0.0299999999999999 0 rpy=-1.5707963267949 -0.00858284690216311 1.57079632679489 -> xyz=0 0.03 0 rpy=-1.5708 -0.91526 1.5708; parent back_left_wheel_axel -> back_right_wheel_axel

Commit message: RAUT-2 #time 10d initial ar tag work

File: rover/src/owr_numbat_tf/robots/owr_numbat_tf.urdf (robot description, URDF)
Before this commit: robot owr_numbat_tf, 13 links, 12 joints
Links:
- added link camera_frame, mass 0.229160254803044; collision box size=0.05 0.05 0.025; visual box size=0.05 0.05 0.025
Joints:
- added joint camera_frame_base: type fixed, parent rover_model, child camera_frame, origin xyz=-0.19 -0.67 0.47 rpy=-4.0766001685455E-16 2.71143453751384E-15 -3.14214183115679, axis 0 0 0

Commit message: RAUT-2 #time 2h added camera stl to numbat urdf file

File: rover/src/owr_numbat_tf/robots/owr_numbat_tf.urdf (robot description, URDF)
Before this commit: robot owr_numbat_tf, 14 links, 13 joints
Links:
- link camera_frame: geometry collision mesh filename=package://owr_numbat_tf/meshes/camera.STL; visual mesh filename=package://owr_numbat_tf/meshes/camera.STL

Commit message: RAUT-2 #time 1h changed camera's frame name and axis in urdf file

File: rover/src/owr_numbat_tf/robots/owr_numbat_tf.urdf (robot description, URDF)
Before this commit: robot owr_numbat_tf, 14 links, 13 joints
Links:
- removed link camera_frame
- added link camera_link, mass 0.229160254803044; collision mesh filename=package://owr_numbat_tf/meshes/camera.STL; visual mesh filename=package://owr_numbat_tf/meshes/camera.STL
Joints:
- joint camera_frame_base: child camera_frame -> camera_link; origin xyz=-0.19 -0.67 0.47 rpy=-4.0766001685455E-16 2.71143453751384E-15 -3.14214183115679 -> xyz=-0.19 -0.67 0.47 rpy=-1.57079632679 0 1.57079632679

Commit message: LR-32 #time 5h converted ar tags message to an odometry message and got the ekf to produce values

File: rover/src/owr_numbat_tf/robots/owr_numbat_tf.urdf (robot description, URDF)
Before this commit: robot owr_numbat_tf, 13 links, 12 joints
Links:
- added link camera_link, mass 0.229160254803044; collision mesh filename=package://owr_numbat_tf/meshes/camera.STL; visual mesh filename=package://owr_numbat_tf/meshes/camera.STL
Joints:
- added joint camera_frame_base: type fixed, parent rover_model, child camera_link, origin xyz=-0.19 -0.67 0.47 rpy=-1.57079632679 0 1.57079632679, axis 0 0 0

Commit message: LR-32 #time 2h changed 2 ar tag localisation code

File: rover/src/owr_numbat_tf/robots/owr_numbat_tf.urdf (robot description, URDF)
Before this commit: robot owr_numbat_tf, 14 links, 13 joints
Links:
- removed link camera_link
- added link ar_camera_link_1, mass 0.229160254803044; collision mesh filename=package://owr_numbat_tf/meshes/camera.STL; visual mesh filename=package://owr_numbat_tf/meshes/camera.STL
- added link ar_camera_link_2, mass 0.229160254803044; collision mesh filename=package://owr_numbat_tf/meshes/camera.STL; visual mesh filename=package://owr_numbat_tf/meshes/camera.STL
Joints:
- removed joint camera_frame_base
- added joint ar_camera_frame_base_1: type fixed, parent rover_model, child ar_camera_link_1, origin xyz=-0.19 -0.67 0.47 rpy=-1.57 0 1.57, axis 0 0 0
- added joint ar_camera_frame_base_2: type fixed, parent rover_model, child ar_camera_link_2, origin xyz=0.19 -0.67 0.47 rpy=-1.57 0 -1.57, axis 0 0 0

Commit message: LR-32 #time 2 h added launch file to start all nodes and camera calibration

File: rover/src/owr_numbat_tf/robots/owr_numbat_tf.urdf (robot description, URDF)
Before this commit: robot owr_numbat_tf, 15 links, 14 joints
Links:
- added link ar_camera_link_3, mass 0.229160254803044; collision mesh filename=package://owr_numbat_tf/meshes/camera.STL; visual mesh filename=package://owr_numbat_tf/meshes/camera.STL
Joints:
- added joint ar_camera_frame_base_3: type fixed, parent rover_model, child ar_camera_link_3, origin xyz=-0.19 -0.67 0.47 rpy=-1.57 0 -1.57, axis 0 0 0
- joint ar_camera_frame_base_1: origin xyz=-0.19 -0.67 0.47 rpy=-1.57 0 1.57 -> xyz=-0.19 -0.67 0.47 rpy=-1.57 0 2.356
- joint ar_camera_frame_base_2: origin xyz=0.19 -0.67 0.47 rpy=-1.57 0 -1.57 -> xyz=-0.19 -0.67 0.47 rpy=-1.57 0 0.785
